Commit message: Things build.

File: urdf/3dof_leg.urdf (robot description, URDF)
Before this commit: robot leg3dof, 5 links, 4 joints
Joints:
- joint joint1: limit (none) -> lower=-3.14 upper=3.14 effort=1 velocity=1
- joint joint2: limit (none) -> lower=-3.14 upper=3.14 effort=1 velocity=1
- joint joint3: limit (none) -> lower=-3.14 upper=3.14 effort=1 velocity=1

Commit message: URDF dimensions should be right.

File: urdf/3dof_leg.urdf (robot description, URDF)
Before this commit: robot leg3dof, 5 links, 4 joints
Links:
- removed link base
Joints:
- removed joint foot_fixed
- joint joint1: axis 0 0 1 -> 1 0 0; child link1 -> link2; origin xyz=0 0 0 rpy=0 0 0 -> xyz=0.2235 0.04241 0 rpy=0 0 0; parent base -> link1
- joint joint2: child link2 -> link3; origin xyz=0 0 -0.2 rpy=0 0 0 -> xyz=0.19425 0.069 0 rpy=0 0 0; parent link1 -> link2
- joint joint3: child link3 -> foot; origin xyz=0 0 -0.2 rpy=0 0 0 -> xyz=0.140 0 0 rpy=0 0 0; parent link2 -> link3
