Commit message: Made a working inverse kinematics control loop in python.

File: urdf/leg3dof.urdf (robot description, URDF)
Before this commit: robot leg3dof, 5 links, 4 joints
Joints:
- joint joint1: limit lower=-3.14 upper=3.14 effort=1 velocity=1 -> (none); type revolute -> continuous
- joint joint2: limit lower=-3.14 upper=3.14 effort=1 velocity=1 -> (none); type revolute -> continuous
- joint joint3: limit lower=-3.14 upper=3.14 effort=1 velocity=1 -> (none); type revolute -> continuous

Commit message: Changed joints to revolute in urdf. Added vizualization to ik script. Changed loading of visual models to not have floating base.

File: urdf/leg3dof.urdf (robot description, URDF)
Before this commit: robot leg3dof, 5 links, 4 joints
Joints:
- joint joint1: limit (none) -> lower=-3.14 upper=3.14 effort=1 velocity=1; type continuous -> revolute
- joint joint2: limit (none) -> lower=-3.14 upper=3.14 effort=1 velocity=1; type continuous -> revolute
- joint joint3: limit (none) -> lower=-3.14 upper=3.14 effort=1 velocity=1; type continuous -> revolute

Commit message: Fixed urdf to be a left leg. Able to load it in pybullet.

File: urdf/leg3dof.urdf (robot description, URDF)
Before this commit: robot leg3dof, 5 links, 4 joints
Links:
- removed link link1
- removed link link2
- removed link link3
- added link calf; visual box size=0.05 0.05 0.19425
- added link hip; visual box size=0.05 0.05 0.05
- added link thigh; visual box size=0.2235 0.05 0.05
- link foot: geometry visual box size=0.05 0.05 0.140
Joints:
- removed joint joint1
- removed joint joint2
- removed joint joint3
- added joint hip_pitch: type revolute, parent thigh, child calf, origin xyz=0.2235 0.04241 0 rpy=0 0 0, axis 0 1 0, limit lower=-3.14 upper=3.14 effort=1 velocity=1
- added joint hip_roll: type revolute, parent hip, child thigh, origin xyz=0 0 0 rpy=0 0 0, axis 1 0 0, limit lower=-3.14 upper=3.14 effort=1 velocity=1
- added joint knee_pitch: type revolute, parent calf, child foot, origin xyz=0 0.069 -0.19425 rpy=0 0 0, axis 0 1 0, limit lower=-3.14 upper=3.14 effort=1 velocity=1
- joint footToToe: origin xyz=0.140 0 0 -> xyz=0 0 -0.140
