Commit message: Have basic quad walking in simulator.

File: urdf/basic_quad.urdf (robot description, URDF)
Before this commit: robot basic_quad, 13 links, 12 joints
Links:
- link bl_calf: geometry collision box size=0.05 0.05 0.19625; visual box size=0.05 0.05 0.19625
- link bl_foot: geometry collision box size=0.05 0.05 0.14; visual box size=0.05 0.05 0.14
- link bl_thigh: geometry collision box size=0.2255 0.05 0.05; visual box size=0.2255 0.05 0.05
- link body: geometry collision box size=0.7 0.25145 0.05; visual box size=0.7 0.25145 0.05
- link br_calf: geometry collision box size=0.05 0.05 0.19625; visual box size=0.05 0.05 0.19625
- link br_foot: geometry collision box size=0.05 0.05 0.14; visual box size=0.05 0.05 0.14
- link br_thigh: geometry collision box size=0.2255 0.05 0.05; visual box size=0.2255 0.05 0.05
- link fl_calf: geometry collision box size=0.05 0.05 0.19625; visual box size=0.05 0.05 0.19625
- link fl_foot: geometry collision box size=0.05 0.05 0.14; visual box size=0.05 0.05 0.14
- link fl_thigh: geometry collision box size=0.2255 0.05 0.05; visual box size=0.2255 0.05 0.05
- link fr_calf: geometry collision box size=0.05 0.05 0.19625; visual box size=0.05 0.05 0.19625
- link fr_foot: geometry collision box size=0.05 0.05 0.14; visual box size=0.05 0.05 0.14
- link fr_thigh: geometry collision box size=0.2255 0.05 0.05; visual box size=0.2255 0.05 0.05

File: urdf/basic_quad.urdf.xacro (robot description, xacro)
@@ -22,4 +22,10 @@
             </material>
         </visual>
+        <collision>
+            <origin xyz="${visual_origin}" rpy="0 0 0"/>
+            <geometry>
+                <box size="${visual_size}"/>
+            </geometry>
+        </collision>
     </link>
 </xacro:macro>

Commit message: Fixed control code and urdf for reversed hip joints. Created seperate requirements.txt for development only utils. Moved sim code so it can see ipc file.

File: urdf/basic_quad.urdf (robot description, URDF)
Before this commit: robot basic_quad, 13 links, 12 joints
Joints:
- joint bl_hip_roll: axis -1 0 0 -> 1 0 0
- joint fr_hip_roll: axis 1 0 0 -> -1 0 0

File: urdf/basic_quad.urdf.xacro (robot description, xacro)
@@ -39,5 +39,5 @@
     </joint>
 </xacro:macro>
-<xacro:macro name="leg3dof" params="prefix parent hip_origin ysign xsign">
+<xacro:macro name="leg3dof" params="prefix parent hip_origin ysign xsign hip_roll_sign">
     <xacro:box_link
         name="${prefix}_thigh"
@@ -57,5 +57,5 @@
         child="${prefix}_thigh"
         origin="${hip_origin}"
-        axis="${xsign * 1} 0 0"/>
+        axis="${hip_roll_sign * 1} 0 0"/>
     <xacro:revolute_joint
         name="${prefix}_hip_pitch"
@@ -82,5 +82,6 @@
     hip_origin="${leg_fb - thigh_length} ${leg_lr} 0.0"
     ysign="1"
-    xsign="1"/>
+    xsign="1"
+    hip_roll_sign="1"/>
 <xacro:leg3dof
     prefix="fr"
@@ -88,5 +89,6 @@
     hip_origin="${leg_fb - thigh_length} ${-leg_lr} 0.0"
     ysign="-1"
-    xsign="1"/>
+    xsign="1"
+    hip_roll_sign="-1"/>
 <xacro:leg3dof
     prefix="bl"
@@ -94,5 +96,6 @@
     hip_origin="${-leg_fb + thigh_length} ${leg_lr} 0.0"
     ysign="1"
-    xsign="-1"/>
+    xsign="-1"
+    hip_roll_sign="1"/>
 <xacro:leg3dof
     prefix="br"
@@ -100,4 +103,5 @@
     hip_origin="${-leg_fb + thigh_length} ${-leg_lr} 0.0"
     ysign="-1"
-    xsign="-1"/>
+    xsign="-1"
+    hip_roll_sign="-1"/>
 </robot>
